File: hardware/DoorControlModule/DoorControlModule.kicad_sch (KiCad schematic)
At the start: 135 parts, among them IC1 CY8C4147AZE-S475, IC2 TLS850B0TBV50ATMA1, IC3 TJA1043T,118, IC4 MAX6818, IC5 LM2901BYPT, IC6 BTS72002EPAXUMA1, IC7 LM74610, J1 501331-0507, J2 64334-0100, Q1 VOMA618A-4X001T, Q2 VOMA618A-4X001T, Q3 IPD50N04S4L08ATMA1, U0 BTM9021EP, U1 BTM9021EP, U2 BTM9021EP, U3 BTN7030_1EPA, U4 BTN7030_1EPA, U5 BTN7030_1EPA, U6 BTN9990LV, U7 BTN9990LV, Y1 CX3225CA24000D0HSSCC, Y2 NX3215SA-32.768K-STD-MUS-2

Commit message: comparator routing updated
Parts:
- removed C56, C57: 100p, Capacitor_SMD:C_0603_1608Metric_Pad1.08x0.95mm_HandSolder, symbol Device:C
- removed D2, D3: LED, LED_SMD:LED_0805_2012Metric_Pad1.15x1.40mm_HandSolder, symbol Device:LED
- removed D8: 33V TVS, Diode_SMD:D_SOD-123, symbol Device:D_TVS
- removed IC2: TLS850B0TBV50ATMA1, SamacSys:TLS850B0TBV33ATMA1, symbol SamacSys:TLS850B0TBV50ATMA1
- removed JP1, JP2: SolderJumper_2_Open, Jumper:SolderJumper-2_P1.3mm_Open_RoundedPad1.0x1.5mm, symbol Jumper:SolderJumper_2_Open
- removed RN10, RN3: 2k0, SamacSys:CAY1647R0F4LF, symbol SamacSys:CAY16-22R0F4LF
- removed U3, U4, U5: BTN7030_1EPA, SamacSys:SOP65P600X115-15N-V, symbol SamacSys:BTN7030-1EPA
- added D10, D9: 3V Z, Diode_SMD:D_SOD-323_HandSoldering, symbol Device:D_Zener
- added D2: ESDA6V1BC6, Package_TO_SOT_SMD:SOT-23-6, symbol Power_Protection:ESDA6V1BC6
- added D3: SMAJ28A, Diode_SMD:D_SMA, symbol Diode:SMAJ28A
- added IC2: TLS850B0TBV33ATMA1, TLS850B0TBV33ATMA1, symbol SamacSys:TLS850B0TBV33ATMA1
- added R33: 2k2, Resistor_SMD:R_0603_1608Metric_Pad0.98x0.95mm_HandSolder, symbol Device:R
- added R34: 2k, Resistor_SMD:R_0603_1608Metric_Pad0.98x0.95mm_HandSolder, symbol Device:R
- added RN13, RN14, RN3: 2k0, SamacSys:CAY16220J2LF, symbol SamacSys:CAY16-220J2LF
- added U3, U4, U5: BTN70301EPAXUMA1, SOP65P600X115-15N-V, symbol SamacSys:BTN70301EPAXUMA1
- J2: footprint SamacSys:643340100 -> SamacSys:64334_JO32_2
- R1: value 2k2 -> 10R
- R10, R9: value 60R -> 2k
- R2: value 1k2 -> DNP
- R32: value 10R -> 2k2
Connections:
- net DIO_4 is gone; now on net ID_2: IC1.58 (P1.0)
- net DIO_4_ is gone; now on net ID_1: R26.1
- net digital_io_3 is gone; now on net digital_io_2: J2.A4
- net +12V: now also IC2.1 (I), IC2.2 (EN), U3.15 (VS), U4.15 (VS), U5.15 (VS)
- net +5V: now also D2.1 (TVS1), IC2.5 (Q); no longer J1.6 (MP_1), J1.7 (MP_2)
- net +BATT: now also D3.1 (A1)
- net AI_5: now also D10.1 (K), R33.2
- net AI_5_: now also R33.1
- net AI_6: now also R32.2, D9.1 (K)
- net AI_6_: now also R32.1
- net DIO_1: now also RN14.4
- net DIO_2: now also RN14.3
- net EN_1: now also RN3.1
- net EN_1_: now also Q1.1 (A), RN3.4; no longer Q2.1 (A)
- net EN_2: now also RN3.2
- net EN_2_: now also Q2.1 (A), RN3.3; no longer Q1.1 (A)
- net Earth: now also J2.X1, J2.X2, R1.1; no longer R32.1
- net GND: now also J1.6 (MP_1), J1.7 (MP_2), J2.C3, R1.2, R2.2, R26.2, D10.2 (A), D2.2 (COM), D2.5 (COM), D3.2 (A2), D9.2 (A), IC2.3 (GND), IC2.6 (TAB), U3.12 (GND_1), U3.13 (GND_2), U3.14 (GND_3), U4.12 (GND_1), U4.13 (GND_2), U4.14 (GND_3), U5.12 (GND_1), U5.13 (GND_2), U5.14 (GND_3); no longer R32.2
- net HB_1_DEN_: now also U4.3 (DEN)
- net HB_1_EN_: now also U4.2 (EN)
- net HB_1_IN_: now also U4.6 (IN)
- net HB_2_DEN_: now also U3.3 (DEN)
- net HB_2_EN_: now also U3.2 (EN)
- net HB_2_IN_: now also U3.6 (IN)
- net MM_DEN_: now also U5.3 (DEN)
- net MM_EN_: now also U5.2 (EN)
- net MM_IN_: now also U5.6 (IN)
- net PWS_RIGHT_DOWN: now also IC4.5 (IN4); no longer IC4.2 (IN1)
- net PWS_RIGHT_DOWN_DEB: now also IC1.23 (P3.5), IC4.16 (OUT4); no longer IC1.18 (P3.0), IC4.19 (OUT1)
- net PWS_RIGHT_LOCK_DOWN: now also IC4.4 (IN3); no longer IC4.3 (IN2)
- net PWS_RIGHT_LOCK_DOWN_DEB: now also IC1.22 (P3.4), IC4.17 (OUT3); no longer IC1.19 (P3.1), IC4.18 (OUT2)
- net PWS_RIGHT_LOCK_UP: now also IC4.2 (IN1); no longer IC4.5 (IN4)
- net PWS_RIGHT_LOCK_UP_DEB: now also IC1.18 (P3.0), IC4.19 (OUT1); no longer IC1.23 (P3.5), IC4.16 (OUT4)
- net PWS_RIGHT_UP: now also IC4.3 (IN2); no longer IC4.4 (IN3)
- net PWS_RIGHT_UP_DEB: now also IC1.19 (P3.1), IC4.18 (OUT2); no longer IC1.22 (P3.4), IC4.17 (OUT3)
- net SWD_CLK: now also D2.4 (TVS3), RN13.4; no longer J1.4
- net SWD_DATA: now also D2.3 (TVS2), RN13.3; no longer J1.5
- net VCC_COMP: now also C53.1, IC5.3 (VCC+)
- net XRES: now also D2.6 (TVS4), R34.1; no longer J1.3
- net digital_io_1: now also RN14.1
- net digital_io_2: now also RN14.2; no longer J2.B3
- net door_lock_sensor_locking: now also J2.B3; no longer J2.C3
- net half_bridge_1: now also U4.10 (OUT_3), U4.8 (OUT_1), U4.9 (OUT_2)
- net half_bridge_2: now also U3.10 (OUT_3), U3.8 (OUT_1), U3.9 (OUT_2)
- net mirror_motor_left_up: now also U5.10 (OUT_3), U5.8 (OUT_1), U5.9 (OUT_2)
- net power_window_switch_down_right: now also J2.A1, RN9.5, RN9.6; no longer J2.A2, RN9.7, RN9.8
- net power_window_switch_up_right: now also J2.A2, RN9.7, RN9.8; no longer J2.A1, RN9.5, RN9.6
- net variable_resistor_high: no longer R26.2
- net at R14.2, R15.2: now also U3.4 (IS), U4.4 (IS), U5.4 (IS)
- net ID_2: now reaches R2.1
- net DIO_3 renamed ID_1
- net VDD_COMP renamed VDD_DEB
- net VDD_DEB: no longer C53.1, IC5.3 (VCC+)
- new net: J1.3, R34.2
- new net: J1.4, RN13.1
- new net: J1.5, RN13.2
- no-connect marks 19 -> 22
Other:
- moved on the sheet: C26, C27, C28, C34, C44, C45, C46, C51, J1, R26, R31, TP1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
