File: hardware/DoorControlModule/DoorControlModule.kicad_sch (KiCad schematic)
At the start: 135 parts, among them IC1 CY8C4147AZE-S475, IC2 TLS850B0TBV33ATMA1, IC3 TJA1043T,118, IC4 MAX6818, IC5 LM2901BYPT, IC6 BTS72002EPAXUMA1, IC7 LM74610, J1 501331-0507, J2 64334-0100, Q1 VOMA618A-4X001T, Q2 VOMA618A-4X001T, Q3 IPD50N04S4L08ATMA1, U0 BTM9021EP, U1 BTM9021EP, U2 BTM9021EP, U3 BTN70301EPAXUMA1, U4 BTN70301EPAXUMA1, U5 BTN70301EPAXUMA1, U6 BTN9990LV, U7 BTN9990LV, Y1 CX3225CA24000D0HSSCC, Y2 NX3215SA-32.768K-STD-MUS-2

Commit message: PCB outline fixed, DRC resolving stage
Parts:
- IC2: footprint TLS850B0TBV33ATMA1 -> SamacSys:TLS850B0TBV33ATMA1
- R2: now left out of the parts list
- U4: renamed from U3; footprint SOP65P600X115-15N-V -> SamacSys:SOP65P600X115-15N-V
- U5: renamed from U4; footprint SOP65P600X115-15N-V -> SamacSys:SOP65P600X115-15N-V
- U6: renamed from U5; footprint SOP65P600X115-15N-V -> SamacSys:SOP65P600X115-15N-V
- renumbered C5 to C10, C13 to C11, C15 to C12, C17 to C13, C12 to C14, C14 to C15, C11 to C17, C21 to C20, C20 to C21, C36 to C35, C38 to C36, C35 to C37, C37 to C38, C42 to C41, C41 to C42, C46 to C44, C44 to C45, C45 to C46, C8 to C5, C53 to C51, C51 to C52, C52 to C53, C9 to C6, C6 to C7, C7 to C8, C10 to C9, D10 to D2, D4 to D3, D9 to D4, D2 to D5, D5 to D6, D6 to D7, D7 to D8, D3 to D9, IC4 to IC3, IC3 to IC4, J2 to J1, J1 to J2, R26 to R1, R9 to R10, R10 to R11, R1 to R12, R31 to R13, R11 to R14, R12 to R15, R13 to R16, R14 to R17, R15 to R18, R16 to R19, R18 to R20, R19 to R21, R20 to R22, R22 to R23, R17 to R24, R21 to R25, R23 to R26, R24 to R27, R32 to R28, R25 to R29, R27 to R30, R28 to R31, R30 to R32, R29 to R33, R33 to R34, R34 to R9, RN2 to RN1, RN9 to RN10, RN14 to RN11, RN11 to RN12, RN12 to RN13, RN1 to RN2, RN13 to RN4, RN4 to RN5, RN5 to RN6, RN6 to RN7, RN7 to RN8, RN8 to RN9, U0 to U1, U1 to U2, U2 to U3, U6 to U7, U7 to U8
Connections:
- net +5V renamed +3.3V

Commit message: top silkscreen cleanup, GND test-point removed
Parts:
- removed TP2: TestPoint, TestPoint:TestPoint_Pad_D1.0mm, symbol Connector:TestPoint
Changed lines of the file:
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@@
-	)
-	(symbol
-		(lib_id "Connector:TestPoint")
-		(at 144.78 76.2 180)
-		(unit 1)
-		(body_style 1)
-		(exclude_from_sim no)
-		(in_bom yes)
-		(on_board yes)
-		(in_pos_files yes)
-		(dnp no)
-		(fields_autoplaced yes)
-		(property "Reference" "TP2"
-			(at 147.32 78.2319 0)
-			(show_name no)
-			(do_not_autoplace no)
-			(effects
-				(font
-					(size 1.27 1.27)
-				)
-				(justify right)
-			)
-		)
-		(property "Value" "TestPoint"
-			(at 147.32 80.7719 0)
-			(show_name no)
-			(do_not_autoplace no)
-			(effects
-				(font
-					(size 1.27 1.27)
-				)
-				(justify right)
-			)
-		)
-		(property "Footprint" "TestPoint:TestPoint_Pad_D1.0mm"
-			(at 139.7 76.2 0)
-			(hide yes)
-			(show_name no)
-			(do_not_autoplace no)
-			(effects
-				(font
-					(size 1.27 1.27)
-				)
-			)
-		)
-		(property "Datasheet" ""
-			(at 139.7 76.2 0)
-			(hide yes)
-			(show_name no)
-			(do_not_autoplace no)
-			(effects
-				(font
-					(size 1.27 1.27)
-				)
-			)
-		)
-		(property "Description" "test point"
-			(at 144.78 76.2 0)
-			(hide yes)
-			(show_name no)
-			(do_not_autoplace no)
-			(effects
-				(font
-					(size 1.27 1.27)
-				)
-			)
-		)
-		(pin "1"
-		)
-		(instances
-			(project "DoorControlModule"
-				(path "/75608795-5873-4a14-bd25-c52b0837619a"
-					(reference "TP2")
-					(unit 1)
-				)
-			)
-		)
 	)
 	(symbol
