File: hardware/DoorControlModule/DoorControlModule.kicad_pcb (KiCad board)
At the start: 6 copper layers, 68.5 x 65.5 mm, 135 parts, among them IC1 CY8C4147AZE-S475, IC2 TLS850B0TBV33ATMA1, IC3 TJA1043T,118, IC4 MAX6818, IC5 LM2901BYPT, IC6 BTS72002EPAXUMA1, IC7 LM74610, J1 501331-0507, J2 64334-0100, Q1 VOMA618A-4X001T, Q2 VOMA618A-4X001T, Q3 IPD50N04S4L08ATMA1, U0 BTM9021EP, U1 BTM9021EP, U2 BTM9021EP, U3 BTN70301EPAXUMA1, U4 BTN70301EPAXUMA1, U5 BTN70301EPAXUMA1, U6 BTN9990LV, U7 BTN9990LV, Y1 CX3225CA24000D0HSSCC, Y2 NX3215SA-32.768K-STD-MUS-2

Commit message: routing update
Routing:
- net VDD_DEB: track 0.00 -> 14.5 mm, vias 0 -> 2
